File: OtterScreen.sch (KiCad schematic (older format))
At the start: 26 parts, among them J1 47272-0001, J2 USB-C_Power, U1 5022505191, U2 NE555, U3 DIO5661, U4 DIO5661

Commit message: updated files
Parts:
- J1: symbol 47272-0001:47272-0001 -> OtterScreen-rescue:47272-0001-47272-0001
- R6, R7: value R8 -> 0.8
Changed lines of the file:
@@
 P 2600 4500
 F 0 "R6" H 2670 4546 50  0000 L CNN
-F 1 "R8" H 2670 4455 50  0000 L CNN
+F 1 "0.8" H 2670 4455 50  0000 L CNN
 F 2 "Resistor_SMD:R_0805_2012Metric" V 2530 4500 50  0001 C CNN
 F 3 "~" H 2600 4500 50  0001 C CNN
@@
 P 2600 2900
 F 0 "R7" H 2670 2946 50  0000 L CNN
-F 1 "R8" H 2670 2855 50  0000 L CNN
+F 1 "0.8" H 2670 2855 50  0000 L CNN
 F 2 "Resistor_SMD:R_0805_2012Metric" V 2530 2900 50  0001 C CNN
 F 3 "~" H 2600 2900 50  0001 C CNN
@@
 	2850 6550 2850 7100
 $Comp
-L 47272-0001:47272-0001 J1
+L OtterScreen-rescue:47272-0001-47272-0001 J1
 U 1 1 5D31A0E0
 P 8000 3600
