File: OtterScreen.sch (KiCad schematic (older format))
At the start: 33 parts, among them J1 47272-0001, J2 USB-C_Power, U1 5022505191, U2 NE555, U5 AMS1117-3.3

Commit message: updated files
Parts:
- U3, U4: renamed from U?; footprint (none) -> Package_SON:WSON-6-1EP_2x2mm_P0.65mm_EP1x1.6mm
- gave numbers to parts that had none: 2
Changed lines of the file:
@@
 $EndComp
 $Comp
-L pro_box_front_sbc-cache:pro_box_front_sbc-rescue_TPS61160A U?
+L pro_box_front_sbc-cache:pro_box_front_sbc-rescue_TPS61160A U4
 U 1 1 5D724657
 P 1950 3450
-F 0 "U?" H 1950 3725 50  0000 C CNN
+F 0 "U4" H 1950 3725 50  0000 C CNN
 F 1 "TPS61160A" H 1950 3634 50  0000 C CNN
-F 2 "" H 1950 3450 50  0001 C CNN
+F 2 "Package_SON:WSON-6-1EP_2x2mm_P0.65mm_EP1x1.6mm" H 1950 3450 50  0001 C CNN
 F 3 "" H 1950 3450 50  0001 C CNN
 	1    1950 3450
@@
 	2750 3550 2750 4000
 $Comp
-L power:GND #PWR?
+L power:GND #PWR0128
 U 1 1 5D733501
 P 2300 3700
-F 0 "#PWR?" H 2300 3450 50  0001 C CNN
+F 0 "#PWR0128" H 2300 3450 50  0001 C CNN
 F 1 "GND" H 2305 3527 50  0000 C CNN
 F 2 "" H 2300 3700 50  0001 C CNN
@@
 $EndComp
 $Comp
-L Device:C_Small C?
+L Device:C_Small C11
 U 1 1 5D734BD2
 P 1500 3850
-F 0 "C?" H 1592 3896 50  0000 L CNN
+F 0 "C11" H 1592 3896 50  0000 L CNN
 F 1 "220nF" H 1592 3805 50  0000 L CNN
 F 2 "Capacitor_SMD:C_0603_1608Metric" H 1500 3850 50  0001 C CNN
@@
 $EndComp
 $Comp
-L power:GND #PWR?
+L power:GND #PWR0132
 U 1 1 5D734BD9
 P 1500 3950
-F 0 "#PWR?" H 1500 3700 50  0001 C CNN
+F 0 "#PWR0132" H 1500 3700 50  0001 C CNN
 F 1 "GND" H 1505 3777 50  0000 C CNN
 F 2 "" H 1500 3950 50  0001 C CNN
@@
 $EndComp
 $Comp
-L power:GND #PWR?
+L power:GND #PWR0133
 U 1 1 5D73A76D
 P 950 2150
-F 0 "#PWR?" H 950 1900 50  0001 C CNN
+F 0 "#PWR0133" H 950 1900 50  0001 C CNN
 F 1 "GND" H 955 1977 50  0000 C CNN
 F 2 "" H 950 2150 50  0001 C CNN
@@
 $EndComp
 $Comp
-L power:GND #PWR?
+L power:GND #PWR0134
 U 1 1 5D73A77A
 P 2950 2150
-F 0 "#PWR?" H 2950 1900 50  0001 C CNN
+F 0 "#PWR0134" H 2950 1900 50  0001 C CNN
 F 1 "GND" H 2955 1977 50  0000 C CNN
 F 2 "" H 2950 2150 50  0001 C CNN
@@
 LEDC2
 $Comp
-L power:GND #PWR?
+L power:GND #PWR0135
 U 1 1 5D73A78C
 P 2950 2800
-F 0 "#PWR?" H 2950 2550 50  0001 C CNN
+F 0 "#PWR0135" H 2950 2550 50  0001 C CNN
 F 1 "GND" H 2955 2627 50  0000 C CNN
 F 2 "" H 2950 2800 50  0001 C CNN
@@
 PWM
 $Comp
-L power:+5V #PWR?
+L power:+5V #PWR0136
 U 1 1 5D73A798
 P 900 1850
-F 0 "#PWR?" H 900 1700 50  0001 C CNN
+F 0 "#PWR0136" H 900 1700 50  0001 C CNN
 F 1 "+5V" V 915 1978 50  0000 L CNN
 F 2 "" H 900 1850 50  0001 C CNN
@@
 $EndComp
 $Comp
-L pro_box_front_sbc-cache:pro_box_front_sbc-rescue_TPS61160A U?
+L pro_box_front_sbc-cache:pro_box_front_sbc-rescue_TPS61160A U3
 U 1 1 5D73A79E
 P 1950 1900
-F 0 "U?" H 1950 2175 50  0000 C CNN
+F 0 "U3" H 1950 2175 50  0000 C CNN
 F 1 "TPS61160A" H 1950 2084 50  0000 C CNN
-F 2 "" H 1950 1900 50  0001 C CNN
+F 2 "Package_SON:WSON-6-1EP_2x2mm_P0.65mm_EP1x1.6mm" H 1950 1900 50  0001 C CNN
 F 3 "" H 1950 1900 50  0001 C CNN
 	1    1950 1900
@@
 	2750 2000 2750 2450
 $Comp
-L power:GND #PWR?
+L power:GND #PWR0137
 U 1 1 5D73A7B2
 P 2300 2150
-F 0 "#PWR?" H 2300 1900 50  0001 C CNN
+F 0 "#PWR0137" H 2300 1900 50  0001 C CNN
 F 1 "GND" H 2305 1977 50  0000 C CNN
 F 2 "" H 2300 2150 50  0001 C CNN
@@
 $EndComp
 $Comp
-L Device:C_Small C?
+L Device:C_Small C10
 U 1 1 5D73A7B8
 P 1500 2300
-F 0 "C?" H 1592 2346 50  0000 L CNN
+F 0 "C10" H 1592 2346 50  0000 L CNN
 F 1 "220nF" H 1592 2255 50  0000 L CNN
 F 2 "Capacitor_SMD:C_0603_1608Metric" H 1500 2300 50  0001 C CNN
@@
 $EndComp
 $Comp
-L power:GND #PWR?
+L power:GND #PWR0145
 U 1 1 5D73A7BF
 P 1500 2400
-F 0 "#PWR?" H 1500 2150 50  0001 C CNN
+F 0 "#PWR0145" H 1500 2150 50  0001 C CNN
 F 1 "GND" H 1505 2227 50  0000 C CNN
 F 2 "" H 1500 2400 50  0001 C CNN
