File: USB-C/USB-C-Screen-Adapter/USB-C-Screen-Adapter.kicad_pcb (KiCad board)
At the start: 4 copper layers, 20.6 x 40 mm, 66 parts, among them J1 USB_C_Receptacle, P1 TC2030-CTX-Tag-Connect, Q1 2N7002, Q2 2N7002, SW1 DFU, U1 SY7200AABC, U2 SY7200AABC, U3 STM32F072CBUx, U4 AP2204R-3.3, U5 USBLC6-4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

Commit message: redone layout
Parts:
- moved R10 68.8 mm to (178.4, 108.7)
- moved R17 68.8 mm to (193.7, 95.1)
- moved R9 68.8 mm to (176.5, 108.7)
- moved D3 48.8 mm to (159.8, 89.2), turned to 270 degrees
- moved D4 46.7 mm to (158.3, 89.2), turned to 270 degrees
- moved C19 44.3 mm to (101.6, 110.3), turned to 270 degrees
- moved R11 42.3 mm to (101.6, 112.2), turned to 270 degrees
- moved Q1 39.2 mm to (122.5, 109.9)
- moved C10 37.3 mm to (123.3, 112.1), turned to 0 degrees
- moved R2 34.1 mm to (129.4, 111.4), turned to 0 degrees
- moved C22 33.3 mm to (127.2, 111.3), turned to 0 degrees
- moved C17 33.2 mm to (135.0, 119.6), turned to 270 degrees
- moved C21 32.1 mm to (134.7, 115.2), turned to 180 degrees
- moved FB1 31.3 mm to (135.2, 117.2), turned to 270 degrees
- moved SW1 29.1 mm to (137.9, 115.6)
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Routing:
- net +3V3: track 0.00 -> 51.7 mm, vias 0 -> 8
- net NRST: track 0.00 -> 39.7 mm, vias 0 -> 2
- net STM_HPD: track 2.43 -> 38.7 mm, vias 0 -> 2
- net SWDIO: track 0.00 -> 26.6 mm
- net SWCLK: track 0.00 -> 25.7 mm
- net L2_P: track 34.1 -> 11.1 mm
- net L2_N: track 31.9 -> 12.1 mm
- net USB_P: track 10.3 -> 29.4 mm, vias 2 -> 1
- net /_L0_N: track 29.0 -> 10.7 mm, vias 2 -> 0
- net /_L0_P: track 28.7 -> 10.7 mm, vias 2 -> 0
- net /_L3_P: track 32.5 -> 14.5 mm
- net /_L3_N: track 33.3 -> 15.3 mm
- net USB_N: track 17.0 -> 34.6 mm, vias 3 -> 4
- net L1_P: track 36.5 -> 19.0 mm
- net L1_N: track 36.6 -> 19.7 mm
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- added copper zone on B.Cu, net +3V3
- added copper zone on F.Cu, net +3V3
Other:
- board size 20.6 x 40 mm -> 40 x 20.8 mm
- net class Default: clearance 0.2 -> 0.13
- net class diff: clearance 0.2 -> 0.13
- rule trace_clearance: 0.2 -> 0.13

Commit message: finalized layout
Parts:
- removed H1, H2: MountingHole_Pad, MountingHole:MountingHole_3.2mm_M3
- moved R17 60.6 mm to (138.0, 119.0)
- moved R9 59.2 mm to (118.2, 119.3)
- moved R10 58.0 mm to (120.7, 114.5), turned to 0 degrees
- moved R8 29.2 mm to (122.8, 112.8)
- moved R5 28.0 mm to (139.1, 109.8), turned to 270 degrees
- moved D4 27.5 mm to (137.6, 107.3)
- moved D3 27.5 mm to (139.1, 107.3)
- moved R13 24.3 mm to (136.7, 111.2)
- moved R14 21.5 mm to (136.1, 109.8), turned to 270 degrees
- moved R16 19.3 mm to (138.1, 111.7), turned to 270 degrees
- moved R12 18.1 mm to (137.6, 109.8), turned to 270 degrees
- moved R7 1.50 mm to (124.3, 111.1)
- moved R2 1.35 mm to (128.1, 111.3)
- moved FB1 1.14 mm to (134.2, 117.7)
- moved C22 1.10 mm to (126.1, 111.3)
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Routing:
- net +3V3: track 51.7 -> 114.2 mm, vias 8 -> 13
- net SBU_ENABLE: track 1.17 -> 56.5 mm, vias 0 -> 4
- net +5V: track 51.8 -> 82.7 mm, vias 7 -> 12
- net CC_TX: track 5.44 -> 25.7 mm, vias 1 -> 2
- net Net-(D3-Pad1): track 0.00 -> 14.3 mm, vias 0 -> 2
- net GND: track 11.7 -> 25.0 mm, vias 5 -> 86
- net USB_N: track 34.6 -> 23.5 mm, vias 4 -> 3
- net Net-(C10-Pad1): track 0.98 -> 10.6 mm, vias 0 -> 2
- net LEDC2: track 18.8 -> 28.3 mm
- net CC_RX: track 2.93 -> 11.2 mm, vias 0 -> 2
- net USB_P: track 29.4 -> 21.2 mm, vias 1 -> 0
- net RXREF: track 0.00 -> 7.92 mm
- net Net-(Q1-Pad2): track 0.00 -> 7.22 mm
- net VBUS_SENSE: track 0.00 -> 6.90 mm
- net CC1: track 20.9 -> 15.9 mm
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- added copper zone on B.Cu, net GND
- added copper zone on F.Cu, net GND
- added copper zone on In1.Cu, net GND
Other:
- net class Default: clearance 0.13 -> 0.1
- net class diff: clearance 0.13 -> 0.1
- net class signal: clearance 0.13 -> 0.1
- rule trace_clearance: 0.13 -> 0.1
- board text added: "Power"
- board text added: "Status"
