File: USB-C-Screen-Adapter-LDR6023SS/USB-C-Screen-Adapter-LDR6023SS.sch (KiCad schematic (older format))
At the start: 40 parts

Commit message: updated schematic
Parts:
- removed C?: 1n, Capacitor_SMD:C_0603_1608Metric, symbol Device:C_Small
- removed C? (x2): 100n, Capacitor_SMD:C_0603_1608Metric, symbol Device:C_Small
- removed D?: D, Diode_SMD:D_SOD-123F, symbol Device:D
- removed R?: 100, Resistor_SMD:R_0603_1608Metric, symbol Device:R
- removed R?: RK14J12R0A09, otter:RK14J12R0A09, symbol otter:RK14J12R0A09
- removed U?: NE555, Package_SO:SO-8_5.3x6.2mm_P1.27mm, symbol Timer:NE555
- added C5, C6, C7, C8: 100n, Capacitor_SMD:C_0402_1005Metric, symbol Device:C_Small
- added R1, R2, R8, R9: 1k, Resistor_SMD:R_0402_1005Metric, symbol Device:R_Small
- added SW1: BRIGHTNESS, otter:K3-2235S-K1, symbol Switch:SW_Push_DPDT
- J2: renamed from J?; footprint (none) -> Connector_PinHeader_2.54mm:PinHeader_1x04_P2.54mm_Vertical
- R6, R7: renamed from R?; value 0.8 -> 1.6
- U3: renamed from U?; footprint (none) -> Package_SO:TSSOP-16_4.4x5mm_P0.65mm
- gave numbers to parts that had none: 29
Connections:
- net GND: now also R1.1, R2.1
- net L0_N: now also C7.1; no longer J1.A10 (RX2-)
- net L0_P: now also C8.1; no longer J1.A11 (RX2+)
- net L1_N: now also C5.1; no longer J1.B10 (RX1-)
- net L1_P: now also C6.1; no longer J1.B11 (RX1+)
- net LEDC1: now also R9.2; no longer U6.3 (FB)
- net LEDC2: now also R8.2; no longer U5.3 (FB)
- new net: R1.2, SW1.2 (B)
- new net: R2.2, SW1.5 (B)
- new net LEDC1DIM: R9.1, SW1.1 (A), U6.3 (FB)
- new net LEDC2DIM: R8.1, SW1.4 (A), U5.3 (FB)
- new net _L0_N: C7.2, J1.A10 (RX2-)
- new net _L0_P: C8.2, J1.A11 (RX2+)
- new net _L1_N: C5.2, J1.B10 (RX1-)
- new net _L1_P: C6.2, J1.B11 (RX1+)
- no-connect marks 5 -> 3
Other:
- note added: "http://cybuild.blogspot.com/2017/07/blog-post.html\n"
- note removed: "http://cybuild.blogspot.com/2017/07/blog-post.html"
- moved on the sheet: C16, C17, C18, C19, R6, R7

Commit message: updated layout
Connections:
- net LEDC1DIM: now also SW1.4 (A); no longer SW1.1 (A)
- net LEDC2DIM: now also SW1.1 (A); no longer SW1.4 (A)
- net USB_N: now also U4.6 (IO4); no longer U4.1 (IO1)
- net USB_P: now also U4.1 (IO1); no longer U4.6 (IO4)
Changed lines of the file:
@@
 EESchema Schematic File Version 4
+LIBS:USB-C-Screen-Adapter-LDR6023SS-cache
 EELAYER 30 0
 EELAYER END
@@
 Text GLabel 5050 6750 0    50   Input ~ 0
 CC2
-Text GLabel 8200 5600 0    50   Input ~ 0
+Text GLabel 8800 5700 2    50   Input ~ 0
 USB_N
 Text GLabel 8450 5050 0    50   Input ~ 0
@@
 	1    0    0    -1
 $EndComp
-Text GLabel 8800 5700 2    50   Input ~ 0
+Text GLabel 8200 5600 0    50   Input ~ 0
 USB_P
 Text GLabel 8450 4950 0    50   Input ~ 0
@@
 Text GLabel 9650 2650 3    50   Input ~ 0
 LEDC1DIM
+Text GLabel 8700 3750 2    50   Input ~ 0
+LEDC1DIM
 Text GLabel 8700 3350 2    50   Input ~ 0
-LEDC1DIM
-Text GLabel 8700 3750 2    50   Input ~ 0
 LEDC2DIM
 $Comp
